File: hardware/KiCad project/key-matrix.kicad_sch (KiCad schematic)
At the start: 134 parts, among them SW1 GRV, SW10 #9, SW11 #0, SW12 -_, SW13 =+, SW14 BCKSPC, SW15 PG-UP, SW16 TAB, SW17 Q, SW18 W, SW19 E, SW2 #1, SW20 R, SW21 T, SW22 Y, SW23 U, SW24 I, SW25 O, SW26 P, SW27 [{, SW28 ]}, SW29 \|, SW3 #2, SW30 PG-DN, SW31 CAPSLOCK, SW32 A, SW33 S, SW34 D, SW35 F, SW36 G, SW37 H, SW38 J, SW39 K, SW4 #3, SW40 L, SW41 ;:, SW42 '", SW44 ENTER, SW45 INS, SW46 LSHIFT, SW47 Z, SW48 X, SW49 C, SW5 #4, SW50 V, SW51 B, SW52 N, SW53 M, SW54 ,<, SW55 >., SW56 /?, SW58 RSHIFT, SW59 UP, SW6 #5, SW60 DEL, SW61 LCTRL, SW62 LALT, SW63 LCOM, SW67 SPACE, SW7 #6, SW71 RCOM, SW72 RALT, SW73 LEFT, SW74 DOWN, SW75 RIGHT, SW8 #7, SW9 #8

Commit message: Added schematic and updated the PCB.
Added the schematics in .jpeg form for easier access along side a new 3D render photo of the keyboard plus a new update to the PCB.
Other:
- company: (none) -> Black Mesa Research Facility
- title: (none) -> InnoKB-x1
Changed lines of the file:
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@@
 	(generator_version "8.0")
 	(paper "A4")
+	(title_block
+		(title "InnoKB-x1")
+		(date "2024-05-13")
+		(rev "0")
+		(company "Black Mesa Research Facility")
+	)
 	(junction
 		(at 217.17 46.99)

Commit message: Finished the PCB design
Parts:
- SW67: footprint Button_Switch_Keyboard:SW_Matias_6.25u -> Button_Switch_Keyboard:SW_Cherry_MX_6.25u_PCB
Changed lines of the file:
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@@
 			)
 		)
-		(property "Footprint" "Button_Switch_Keyboard:SW_Matias_6.25u"
+		(property "Footprint" "Button_Switch_Keyboard:SW_Cherry_MX_6.25u_PCB"
 			(at 129.54 128.27 0)
 			(effects
