File: hardware/KiCad project/keyboard.kicad_pcb (KiCad board)
At the start: 2 copper layers, 362 x 154.9 mm, 155 parts, among them J1 USB-C, J2 AVR-ISP-6, K1 SW_MEC_5E, SW1 GRV, SW10 #9, SW11 #0, SW12 -_, SW13 =+, SW14 BCKSPC, SW15 PG-UP, SW16 TAB, SW17 Q, SW18 W, SW19 E, SW2 #1, SW20 R, SW21 T, SW22 Y, SW23 U, SW24 I, SW25 O, SW26 P, SW27 [{, SW28 ]}, SW29 \|, SW3 #2, SW30 PG-DN, SW31 CAPSLOCK, SW32 A, SW33 S, SW34 D, SW35 F, SW36 G, SW37 H, SW38 J, SW39 K, SW4 #3, SW40 L, SW41 ;:, SW42 '", SW44 ENTER, SW45 INS, SW46 LSHIFT, SW47 Z, SW48 X, SW49 C, SW5 #4, SW50 V, SW51 B, SW52 N, SW53 M, SW54 ,<, SW55 >., SW56 /?, SW58 RSHIFT, SW59 UP, SW6 #5, SW60 DEL, SW61 LCTRL, SW62 LALT, SW63 LCOM, SW67 SPACE, SW7 #6, SW71 RCOM, SW72 RALT, SW73 LEFT, SW74 DOWN, SW75 RIGHT, SW8 #7, SW9 #8, U1 ATmega32U4-A, Y1 Crystal_GND24_Small

Commit message: Added schematic and updated the PCB.
Added the schematics in .jpeg form for easier access along side a new 3D render photo of the keyboard plus a new update to the PCB.
Parts:
- R1, R2, R3, R4, R5, R6: footprint Capacitor_SMD:C_0603_1608Metric_Pad1.08x0.95mm_HandSolder -> Capacitor_SMD:C_0805_2012Metric_Pad1.18x1.45mm_HandSolder
- U1: moved to F.Cu
- moved C9 369.1 mm to (643.9, -51.2), turned to 90 degrees
- moved J2 363.9 mm to (646.7, -56.8)
- moved R6 353.0 mm to (622.8, -55.8), turned to 45 degrees
- moved C7 345.6 mm to (610.3, -60.4), turned to 45 degrees
- moved K1 345.5 mm to (628.2, -53.2)
- moved R2 339.6 mm to (618.7, -45.1), turned to 135 degrees
- moved C8 339.6 mm to (615.7, -42.1), turned to -45 degrees
- moved D1 339.1 mm to (633.6, -37.9), turned to 180 degrees
- moved C3 338.4 mm to (620.2, -46.7), turned to 135 degrees
- moved R5 337.3 mm to (604.0, -55.5), turned to 135 degrees
- moved R1 335.8 mm to (617.2, -43.6), turned to 135 degrees
- moved C6 332.4 mm to (605.3, -49.2), turned to -45 degrees
- moved C4 330.8 mm to (610.1, -44.1), turned to 135 degrees
- moved C2 238.2 mm to (621.0, -57.6), turned to 45 degrees
- moved C1 236.3 mm to (619.0, -59.6), turned to 45 degrees
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Routing:
- net COL10: track 0.00 -> 92.6 mm
- net COL1: track 0.00 -> 91.9 mm
- net COL6: track 0.00 -> 90.1 mm
- net COL2: track 0.00 -> 88.9 mm
- net COL13: track 0.00 -> 87.9 mm
- net COL11: track 0.00 -> 87.1 mm
- net COL12: track 0.00 -> 85.1 mm
- net COL0: track 0.00 -> 84.7 mm
- net COL14: track 0.00 -> 77.4 mm
- net COL8: track 0.00 -> 68.4 mm
- net COL7: track 0.00 -> 67.7 mm
- net COL3: track 0.00 -> 67.7 mm
- net COL9: track 0.00 -> 67.7 mm
- net COL5: track 0.00 -> 67.7 mm
- net COL4: track 0.00 -> 67.7 mm
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Other:
- board size 362 x 154.9 mm -> 314.5 x 134.9 mm

Commit message: Finished the PCB design
Parts:
- added REF**: MountingHole_3.2mm_M3_Pad, MountingHole:MountingHole_3.2mm_M3_Pad, F.Cu at (53.8, 206.2)
- added REF**: MountingHole_3.2mm_M3_Pad, MountingHole:MountingHole_3.2mm_M3_Pad, F.Cu at (324.8, 101.5)
- added REF**: MountingHole_3.2mm_M3_Pad, MountingHole:MountingHole_3.2mm_M3_Pad, F.Cu at (53.7, 101.5)
- added REF**: MountingHole_3.2mm_M3_Pad, MountingHole:MountingHole_3.2mm_M3_Pad, F.Cu at (360.0, 206.2)
- moved C9 497.6 mm to (209.5, 191.5), turned to 180 degrees
- moved R6 484.2 mm to (213.5, 203.0), turned to 0 degrees
- moved C5 479.4 mm to (209.5, 196.5), turned to 180 degrees
- moved C3 476.1 mm to (209.5, 194.0), turned to 0 degrees
- moved C7 473.0 mm to (217.5, 203.0), turned to 0 degrees
- moved C2 468.3 mm to (230.3, 200.6), turned to 180 degrees
- moved C1 466.6 mm to (230.3, 198.5), turned to 180 degrees
- moved U1 465.2 mm to (218.9, 194.8), turned to 0 degrees
- moved Y1 465.0 mm to (235.3, 194.5), turned to -90 degrees
- moved C8 461.8 mm to (214.7, 187.0), turned to 0 degrees
- moved C4 454.0 mm to (227.0, 199.5), turned to -90 degrees
- moved R5 450.0 mm to (227.5, 191.0), turned to 0 degrees
- moved C6 449.2 mm to (223.2, 187.0), turned to 180 degrees
- moved J2 351.8 mm to (334.5, 105.5), turned to -90 degrees
- moved D46 329.3 mm to (355.5, 164.5), turned to 0 degrees
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Connections:
- U1 pad 19: COL8 -> COL0
- U1 pad 20: COL9 -> COL1
- U1 pad 21: COL10 -> COL2
- U1 pad 22: COL11 -> COL3
- U1 pad 25: COL12 -> COL14
- U1 pad 27: COL14 -> COL12
- U1 pad 28: COL0 -> COL11
- U1 pad 29: COL1 -> COL10
- U1 pad 30: COL2 -> COL9
- U1 pad 31: COL3 -> COL8
- U1 pad 32: COL4 -> COL7
- U1 pad 39: ROW4 -> ROW2
- U1 pad 41: ROW2 -> ROW4
- U1 pad 8: COL7 -> COL4
Routing:
- net ROW0: track 0.00 -> 383.3 mm, vias 0 -> 15
- net ROW1: track 0.00 -> 344.4 mm, vias 0 -> 15
- net ROW2: track 0.00 -> 319.2 mm, vias 0 -> 14
- net ROW4: track 0.00 -> 294.9 mm, vias 0 -> 10
- net ROW3: track 0.00 -> 293.8 mm, vias 0 -> 14
- net VBUS: track 3.86 -> 267.0 mm, vias 0 -> 2
- net +5V: track 25.6 -> 287.8 mm, vias 0 -> 2
- net ~{RST}: track 3.06 -> 250.6 mm, vias 0 -> 2
- net SCK: track 0.00 -> 236.7 mm, vias 0 -> 2
- net Net-(U1-D-): track 2.59 -> 236.3 mm, vias 0 -> 2
- net MOSI: track 0.00 -> 233.3 mm, vias 0 -> 2
- net Net-(U1-D+): track 2.46 -> 235.4 mm, vias 0 -> 2
- net MISO: track 0.00 -> 232.8 mm, vias 0 -> 2
- net COL2: track 88.9 -> 280.1 mm, vias 0 -> 1
- net COL1: track 91.9 -> 256.8 mm, vias 0 -> 1
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- added copper zone on B.Cu, net GND
- added copper zone on F.Cu, net GND
Other:
- board size 314.5 x 134.9 mm -> 313.3 x 111.7 mm
- board text added: "InnoKB-X1"
- board text added: "Tudor S. {dblquote}Flăcărică{dblquote}"
