File: hardware/KiCad project/keyboard.kicad_sch (KiCad schematic)
At the start: 21 parts, among them J1 USB-C, J2 AVR-ISP-6, K1 SW_MEC_5E, U1 ATmega32U4-A, Y1 Crystal_GND24_Small

Commit message: Added schematic and updated the PCB.
Added the schematics in .jpeg form for easier access along side a new 3D render photo of the keyboard plus a new update to the PCB.
Parts:
- R1, R2, R3, R4, R5, R6: footprint Capacitor_SMD:C_0603_1608Metric_Pad1.08x0.95mm_HandSolder -> Capacitor_SMD:C_0805_2012Metric_Pad1.18x1.45mm_HandSolder
Other:
- company: (none) -> Black Mesa Research Facility
- title: (none) -> InnoKB-x1
Changed lines of the file:
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@@
 	(generator_version "8.0")
 	(paper "A4")
+	(title_block
+		(title "InnoKB-x1")
+		(date "2024-05-13")
+		(rev "0")
+		(company "Black Mesa Research Facility")
+	)
 	(junction
 		(at 222.25 38.1)
@@
 			)
 		)
-		(property "Footprint" "Capacitor_SMD:C_0603_1608Metric_Pad1.08x0.95mm_HandSolder"
+		(property "Footprint" "Capacitor_SMD:C_0805_2012Metric_Pad1.18x1.45mm_HandSolder"
 			(at 204.47 74.93 0)
 			(effects
@@
 			)
 		)
-		(property "Footprint" "Capacitor_SMD:C_0603_1608Metric_Pad1.08x0.95mm_HandSolder"
+		(property "Footprint" "Capacitor_SMD:C_0805_2012Metric_Pad1.18x1.45mm_HandSolder"
 			(at 187.96 49.53 0)
 			(effects
@@
 			)
 		)
-		(property "Footprint" "Capacitor_SMD:C_0603_1608Metric_Pad1.08x0.95mm_HandSolder"
+		(property "Footprint" "Capacitor_SMD:C_0805_2012Metric_Pad1.18x1.45mm_HandSolder"
 			(at 119.38 114.3 0)
 			(effects
@@
 			)
 		)
-		(property "Footprint" "Capacitor_SMD:C_0603_1608Metric_Pad1.08x0.95mm_HandSolder"
+		(property "Footprint" "Capacitor_SMD:C_0805_2012Metric_Pad1.18x1.45mm_HandSolder"
 			(at 119.38 111.76 0)
 			(effects
@@
 			)
 		)
-		(property "Footprint" "Capacitor_SMD:C_0603_1608Metric_Pad1.08x0.95mm_HandSolder"
+		(property "Footprint" "Capacitor_SMD:C_0805_2012Metric_Pad1.18x1.45mm_HandSolder"
 			(at 242.57 100.33 0)
 			(effects
@@
 			)
 		)
-		(property "Footprint" "Capacitor_SMD:C_0603_1608Metric_Pad1.08x0.95mm_HandSolder"
+		(property "Footprint" "Capacitor_SMD:C_0805_2012Metric_Pad1.18x1.45mm_HandSolder"
 			(at 204.47 72.39 0)
 			(effects

Commit message: Finished the PCB design
Connections:
- net COL0: now also U1.19 (PD1); no longer U1.28 (PB4)
- net COL1: now also U1.20 (PD2); no longer U1.29 (PB5)
- net COL10: now also U1.29 (PB5); no longer U1.21 (PD3)
- net COL11: now also U1.28 (PB4); no longer U1.22 (PD5)
- net COL12: now also U1.27 (PD7); no longer U1.25 (PD4)
- net COL14: now also U1.25 (PD4); no longer U1.27 (PD7)
- net COL2: now also U1.21 (PD3); no longer U1.30 (PB6)
- net COL3: now also U1.22 (PD5); no longer U1.31 (PC6)
- net COL4: now also U1.8 (PB0); no longer U1.32 (PC7)
- net COL7: now also U1.32 (PC7); no longer U1.8 (PB0)
- net COL8: now also U1.31 (PC6); no longer U1.19 (PD1)
- net COL9: now also U1.30 (PB6); no longer U1.20 (PD2)
- net ROW2: now also U1.39 (PF4); no longer U1.41 (PF0)
- net ROW4: now also U1.41 (PF0); no longer U1.39 (PF4)
